Commit message: Add velodyne support.

File: p3dx_description/urdf/pioneer3dx.xacro (robot description, xacro)
@@ -45,4 +45,35 @@
 		</collision>
 	</link>
+	<!-- my code starts-->
+<!--
+	<link name="camera">
+    <collision>
+      <origin xyz="0 5 0" rpy="0 0 0"/>
+      <geometry>
+        <box size="0.05 0.05 0.05"/>
+      </geometry>
+    </collision>
+    <visual>
+      <origin xyz="0 0 0" rpy="0 0 0"/>
+      <geometry>
+        <box size="0.05 0.05 0.05"/>
+      </geometry>
+      <material name="green"/>
+    </visual>
+    <inertial>
+      <mass value="0.1" />
+      <origin xyz="0 0 0" rpy="0 0 0"/>
+      <box_inertia m="0.1" x="0.05" y="0.05" z="0.05" />
+      <inertia ixx="1e-6" ixy="0" ixz="0" iyy="1e-6" iyz="0" izz="1e-6" />
+    </inertial>
+  </link>
+  <joint name="camera_joint" type="fixed">
+    <axis xyz="0 1 0" />
+    <origin xyz=".2 0 0" rpy="0 0 0"/>
+    <parent link="top_plate"/>
+    <child link="camera"/>
+  </joint>
+-->
+<!-- my code ends -->
   <!-- top_plate -->
 	<link name="top_plate">
@@ -197,6 +228,5 @@
 		<child link="front_sonar" />
 	</joint>
-	<!-- lms100 laser -->
-	<link name="lms100">
+<!--<link name="lms100">
 		<inertial>
 			<mass value="1e-5" />
@@ -216,10 +246,313 @@
 			</geometry>
 		</collision>
-	</link>
-	<joint name="lms100_joint" type="fixed">
+	</link>-->
+<!--<link name="lidar_base">
+		<inertial>
+			<mass value="1e-5" />
+			<origin xyz="0 0 0" rpy="0 0 0" />
+			<inertia ixx="1e-6" ixy="0" ixz="0" iyy="1e-6" iyz="0" izz="1e-6" />
+		</inertial>
+		<visual>
+			<origin xyz="0 0 0" rpy="0 0 0" />
+			<geometry>
+				<mesh filename="package://p3dx_description/meshes/velodyne_top.dae" />
+			</geometry>
+		</visual>
+		<collision>
+			<origin xyz="0 0 0" rpy="0 0 0" />
+			<geometry>
+				<box size="0.1 0.1 0.1" />
+			</geometry>
+		</collision>
+	</link>-->
+	<!--<joint name="lidar_joint1" type="fixed">
 		<axis xyz="0 1 0" />
 		<origin xyz="0.16 0 0.15" rpy="0 0 0" />
 		<parent link="base_link" />
 		<child link="lms100" />
-	</joint>
+	</joint>-->
+	<!--<joint name="lidar_joint2" type="fixed">
+		<axis xyz="0 1 0" />
+		<origin xyz="0.16 0 0.15" rpy="0 0 0" />
+		<parent link="base_link" />
+		<child link="lms100" />
+	</joint>-->
+	<!-- lms100 laser -->
+	<link name="lidarbase">
+		<inertial>
+			<mass value="1.2" />
+			<origin xyz="0 0 0" rpy="0 0 0" />
+			<inertia ixx="0.001087473" ixy="0" ixz="0" iyy="0.001087473" iyz="0" izz="0.001092437" />
+		</inertial>
+		<visual>
+			<origin xyz="0 0 0" rpy="0 0 0" />
+			<geometry>
+				<mesh filename="package://p3dx_description/meshes/velodyne_base.dae" />
+			</geometry>
+		</visual>
+		<collision>
+			<origin xyz="0 0 0" rpy="0 0 0" />
+			<geometry>
+				<box size="0.1 0.1 0.1" />
+			</geometry>
+		</collision>
+	</link>
+	<link name="lidartop">
+		<inertial>
+			<mass value="1.2" />
+			<origin xyz="0 0 0" rpy="0 0 0" />
+			<inertia ixx="0.001087473" ixy="0" ixz="0" iyy="0.001087473" iyz="0" izz="0.001092437" />
+		</inertial>
+		<visual>
+			<origin xyz="0 0 0" rpy="0 0 0" />
+			<geometry>
+				<mesh filename="package://p3dx_description/meshes/velodyne_top.dae" />
+			</geometry>
+		</visual>
+		<collision>
+			<origin xyz="0 0 0" rpy="0 0 0" />
+			<geometry>
+				<box size="0.1 0.1 0.1" />
+			</geometry>
+		</collision>
+	<sensor type="ray" name="sensor">
+        <pose>0 0 -0.004645 1.5707 0 0</pose>
+        <visualize>true</visualize>
+        <update_rate>30</update_rate>
+        <ray>
+          <noise>
+            <type>gaussian</type>
+            <mean>0.0</mean>
+            <stddev>0.1</stddev>
+          </noise>
+          <scan>
+            <horizontal>
+              <samples>32</samples>
+              <resolution>1</resolution>
+              <min_angle>-0.53529248</min_angle>
+              <max_angle>0.18622663</max_angle>
+            </horizontal>
+          </scan>
+          <range>
+            <min>0.1</min>
+            <max>70</max>
+            <resolution>0.02</resolution>
+          </range>
+        </ray>
+      </sensor>
+	</link>
+	<joint name="lidar_joint" type="fixed">
+		<axis xyz="0 1 0" />
+		<origin xyz="0 0 0" rpy="0 0 0" />
+		<parent link="top_plate" />
+		<child link="lidarbase" />
+	</joint>
+	<joint name="lidar_joint1" type="fixed">
+		<axis xyz="0 1 0" />
+		<origin xyz="0 0 0.05" rpy="0 0 0" />
+		<parent link="top_plate" />
+		<child link="lidartop" />
+	</joint>
+<!-- lidar connection-->
+<!--
+    <link name="base">
+      <pose>0 0 0.029335 0 0 0</pose>
+      <inertial>
+        <mass>1.2</mass>
+        <inertia>
+          <ixx>0.001087473</ixx>
+          <iyy>0.001087473</iyy>
+          <izz>0.001092437</izz>
+          <ixy>0</ixy>
+          <ixz>0</ixz>
+          <iyz>0</iyz>
+        </inertia>
+      </inertial>
+      <collision name="base_collision">
+        <geometry>
+          <cylinder>
+            <radius>.04267</radius>
+            <length>.05867</length>
+          </cylinder>
+        </geometry>
+      </collision>
+      <visual name="base_visual">
+        <pose>0 0 -0.029335 0 0 0</pose>
+        <geometry>
+          <mesh>
+            <uri>model://velodyne_hdl32/meshes/velodyne_base.dae</uri>
+          </mesh>
+        </geometry>
+      </visual>
+    </link>
+    <link name="top">
+      <pose>0 0 0.095455 0 0 0</pose>
+      <inertial>
+        <mass>0.1</mass>
+        <inertia>
+          <ixx>0.000090623</ixx>
+          <iyy>0.000090623</iyy>
+          <izz>0.000091036</izz>
+          <ixy>0</ixy>
+          <ixz>0</ixz>
+          <iyz>0</iyz>
+        </inertia>
+      </inertial>
+      <collision name="top_collision">
+        <geometry>
+          <cylinder>
+            <radius>0.04267</radius>
+            <length>0.07357</length>
+          </cylinder>
+        </geometry>
+      </collision>
+      <visual name="top_visual">
+        <pose>0 0 -0.0376785 0 0 1.5707</pose>
+        <geometry>
+          <mesh>
+            <uri>model://velodyne_hdl32/meshes/velodyne_top.dae</uri>
+          </mesh>
+        </geometry>
+      </visual>
+      <sensor type="ray" name="sensor">
+        <pose>0 0 -0.004645 1.5707 0 0</pose>
+        <visualize>true</visualize>
+        <update_rate>30</update_rate>
+        <ray>
+          <noise>
+            <type>gaussian</type>
+            <mean>0.0</mean>
+            <stddev>0.1</stddev>
+          </noise>
+          <scan>
+            <horizontal>
+              <samples>32</samples>
+              <resolution>1</resolution>
+              <min_angle>-0.53529248</min_angle>
+              <max_angle>0.18622663</max_angle>
+            </horizontal>
+          </scan>
+          <range>
+            <min>0.1</min>
+            <max>70</max>
+            <resolution>0.02</resolution>
+          </range>
+        </ray>
+      </sensor>
+    </link>
+    <joint type="revolute" name="joint">
+      <pose>0 0 -0.036785 0 0 0</pose>
+      <parent link="top_plate"/>
+      <child>top</child>
+      <axis>
+        <xyz>0 0 1</xyz>
+        <limit>
+          <lower>-10000000000000000</lower>
+          <upper>10000000000000000</upper>
+        </limit>
+      </axis>
+    </joint>
+-->
+<!-- lidar connection-->
+<!--my code
+      <link name='base'>
+        <pose frame=''>0 0 0.029335 0 -0 0</pose>
+        <inertial>
+          <mass>1.2</mass>
+          <inertia>
+            <ixx>0.00108747</ixx>
+            <iyy>0.00108747</iyy>
+            <izz>0.00109244</izz>
+            <ixy>0</ixy>
+            <ixz>0</ixz>
+            <iyz>0</iyz>
+          </inertia>
+        </inertial>
+        <collision name='base_collision'>
+          <geometry>
+            <cylinder>
+              <radius>0.04267</radius>
+              <length>0.05867</length>
+            </cylinder>
+          </geometry>
+        </collision>
+        <visual name='base_visual'>
+          <pose frame=''>0 0 -0.029335 0 -0 0</pose>
+          <geometry>
+            <mesh>
+              <uri>model://velodyne_hdl32/meshes/velodyne_base.dae</uri>
+            </mesh>
+          </geometry>
+        </visual>
+      </link>
+      <link name='top'>
+        <pose frame=''>0 0 0.095455 0 -0 0</pose>
+        <inertial>
+          <mass>0.1</mass>
+          <inertia>
+            <ixx>9.0623e-05</ixx>
+            <iyy>9.0623e-05</iyy>
+            <izz>9.1036e-05</izz>
+            <ixy>0</ixy>
+            <ixz>0</ixz>
+            <iyz>0</iyz>
+          </inertia>
+        </inertial>
+        <collision name='top_collision'>
+          <geometry>
+            <cylinder>
+              <radius>0.04267</radius>
+              <length>0.07357</length>
+            </cylinder>
+          </geometry>
+        </collision>
+        <visual name='top_visual'>
+          <pose frame=''>0 0 -0.037679 0 -0 1.5707</pose>
+          <geometry>
+            <mesh>
+              <uri>model://velodyne_hdl32/meshes/velodyne_top.dae</uri>
+            </mesh>
+          </geometry>
+        </visual>
+        <sensor name='sensor' type='ray'>
+          <pose frame=''>0 0 -0.004645 1.5707 -0 0</pose>
+          <visualize>1</visualize>
+          <update_rate>30</update_rate>
+          <ray>
+            <noise>
+              <type>gaussian</type>
+              <mean>0</mean>
+              <stddev>0.1</stddev>
+            </noise>
+            <scan>
+              <horizontal>
+                <samples>32</samples>
+                <resolution>1</resolution>
+                <min_angle>-0.535292</min_angle>
+                <max_angle>0.186227</max_angle>
+              </horizontal>
+            </scan>
+            <range>
+              <min>0.1</min>
+              <max>70</max>
+              <resolution>0.02</resolution>
+            </range>
+          </ray>
+        </sensor>
+      </link>
+      <joint name='joint' type='revolute'>
+        <pose frame=''>0 0 -0.036785 0 -0 0</pose>
+        <parent>base</parent>
+        <child>top</child>
+        <axis>
+          <xyz>0 0 1</xyz>
+          <limit>
+            <lower>-1e+16</lower>
+            <upper>1e+16</upper>
+          </limit>
+          <use_parent_model_frame>0</use_parent_model_frame>
+        </axis>
+      </joint>
+      <pose frame=''>-0.701772 0.531559 0.001683 0 -0 0</pose>
+my code-->
 </robot>

Commit message: Final working model.

File: p3dx_description/urdf/pioneer3dx.xacro (robot description, xacro)
@@ -342,4 +342,6 @@
       </sensor>
 	</link>
+    <link name="laser">
+    </link>
 	<joint name="lidar_joint" type="fixed">
 		<axis xyz="0 1 0" />
@@ -354,4 +356,9 @@
 		<child link="lidartop" />
 	</joint>
+    <joint name="lidar_optical_joint" type="fixed">
+        <origin xyz="0 0 0" rpy="${-pi/2} 0 ${-pi/2}"/>
+        <parent link="lidartop"/>
+        <child link="laser"/>
+    </joint>
 <!-- lidar connection-->
 <!--
